Commit message: updated pos

File: body.urdf (robot description, URDF)
Before this commit: robot robot, 3 links, 2 joints
Joints:
- joint Torso_BackLeg: origin xyz=0 0 0.5 rpy=0 0 0 -> xyz=2 0 1 rpy=0 0 0
- joint Torso_FrontLeg: origin xyz=0 0.5 0.5 rpy=0 0 0 -> xyz=1 0 1 rpy=0 0 0

Commit message: quadruped

File: body.urdf (robot description, URDF)
Before this commit: robot robot, 3 links, 2 joints
Links:
- added link BackLeg2, mass 1; collision box size=0.2 0.2 1; visual box size=0.2 0.2 1
- added link FrontLeg2, mass 1; collision box size=0.2 0.2 1; visual box size=0.2 0.2 1
- added link LeftLeg, mass 1; collision box size=1 0.2 0.2; visual box size=1 0.2 0.2
- added link LeftLeg2, mass 1; collision box size=0.2 0.2 1; visual box size=0.2 0.2 1
- added link RightLeg, mass 1; collision box size=1 0.2 0.2; visual box size=1 0.2 0.2
- added link RightLeg2, mass 1; collision box size=0.2 0.2 1; visual box size=0.2 0.2 1
- link BackLeg: geometry collision box size=0.2 1 0.2; visual box size=0.2 1 0.2
- link FrontLeg: geometry collision box size=0.2 1 0.2; visual box size=0.2 1 0.2
Joints:
- added joint BackLeg_BackLeg2: type revolute, parent BackLeg, child BackLeg2, origin xyz=0 -1 0 rpy=0 0 0, axis 1 0 0, limit lower=-3.14159 upper=3.14159 effort=0.0 velocity=0.0
- added joint FrontLeg_FrontLeg2: type revolute, parent FrontLeg, child FrontLeg2, origin xyz=0 1 0 rpy=0 0 0, axis 1 0 0, limit lower=-3.14159 upper=3.14159 effort=0.0 velocity=0.0
- added joint LeftLeg_LeftLeg2: type revolute, parent LeftLeg, child LeftLeg2, origin xyz=-1 0 0 rpy=0 0 0, axis 0 1 0, limit lower=-3.14159 upper=3.14159 effort=0.0 velocity=0.0
- added joint RightLeg_RightLeg2: type revolute, parent RightLeg, child RightLeg2, origin xyz=1 0 0 rpy=0 0 0, axis 0 1 0, limit lower=-3.14159 upper=3.14159 effort=0.0 velocity=0.0
- added joint Torso_LeftLeg: type revolute, parent Torso, child LeftLeg, origin xyz=-0.5 0 1 rpy=0 0 0, axis 0 1 0, limit lower=-3.14159 upper=3.14159 effort=0.0 velocity=0.0
- added joint Torso_RightLeg: type revolute, parent Torso, child RightLeg, origin xyz=0.5 0 1 rpy=0 0 0, axis 0 1 0, limit lower=-3.14159 upper=3.14159 effort=0.0 velocity=0.0
- joint Torso_BackLeg: axis 0 1 0 -> 1 0 0; origin xyz=2 0 1 rpy=0 0 0 -> xyz=0 -0.5 1 rpy=0 0 0
- joint Torso_FrontLeg: axis 0 1 0 -> 1 0 0; origin xyz=1 0 1 rpy=0 0 0 -> xyz=0 0.5 1 rpy=0 0 0

Commit message: inital final project design

File: body.urdf (robot description, URDF)
Before this commit: robot robot, 9 links, 8 joints
Links:
- removed link BackLeg
- removed link BackLeg2
- removed link FrontLeg
- removed link FrontLeg2
- removed link LeftLeg
- removed link LeftLeg2
- removed link RightLeg
- removed link RightLeg2
- removed link Torso
- added link backleg, mass 1; collision box size=2 0.2 0.5; visual box size=2 0.2 0.5
- added link backleg2, mass 1; collision box size=0.2 0.2 1.5; visual box size=0.2 0.2 1.5
- added link frontleg, mass 1; collision box size=2 0.2 0.5; visual box size=2 0.2 0.5
- added link frontleg2, mass 1; collision box size=0.2 0.2 1.5; visual box size=0.2 0.2 1.5
- added link leftleg, mass 1; collision box size=2 0.2 0.5; visual box size=2 0.2 0.5
- added link leftleg2, mass 1; collision box size=0.2 0.2 1.5; visual box size=0.2 0.2 1.5
- added link rightleg, mass 1; collision box size=2 0.2 0.5; visual box size=2 0.2 0.5
- added link rightleg2, mass 1; collision box size=0.2 0.2 1.5; visual box size=0.2 0.2 1.5
- added link torso, mass 1; collision box size=1 3 0.5; visual box size=1 3 0.5
Joints:
- removed joint BackLeg_BackLeg2
- removed joint FrontLeg_FrontLeg2
- removed joint LeftLeg_LeftLeg2
- removed joint RightLeg_RightLeg2
- removed joint Torso_BackLeg
- removed joint Torso_FrontLeg
- removed joint Torso_LeftLeg
- removed joint Torso_RightLeg
- added joint backleg_backleg2: type revolute, parent backleg, child backleg2, origin xyz=-1.5 -0.25 0 rpy=0 0 0, axis 0 1 0, limit lower=-3.14159 upper=3.14159 effort=0.0 velocity=0.0
- added joint frontleg_frontleg2: type revolute, parent frontleg, child frontleg2, origin xyz=1.5 -0.25 0 rpy=0 0 0, axis 0 1 0, limit lower=-3.14159 upper=3.14159 effort=0.0 velocity=0.0
- added joint leftleg_leftleg2: type revolute, parent leftleg, child leftleg2, origin xyz=-1.5 0.25 0 rpy=0 0 0, axis 0 1 0, limit lower=-3.14159 upper=3.14159 effort=0.0 velocity=0.0
- added joint rightleg_rightleg2: type revolute, parent rightleg, child rightleg2, origin xyz=1.5 0.25 0 rpy=0 0 0, axis 0 1 0, limit lower=-3.14159 upper=3.14159 effort=0.0 velocity=0.0
- added joint torso_backleg: type revolute, parent torso, child backleg, origin xyz=-0.5 -0.5 1 rpy=0 0 0, axis 0 1 0, limit lower=-3.14159 upper=3.14159 effort=0.0 velocity=0.0
- added joint torso_frontleg: type revolute, parent torso, child frontleg, origin xyz=0.5 -0.5 1 rpy=0 0 0, axis 0 1 0, limit lower=-3.14159 upper=3.14159 effort=0.0 velocity=0.0
- added joint torso_leftleg: type revolute, parent torso, child leftleg, origin xyz=-0.5 0.5 1 rpy=0 0 0, axis 0 1 0, limit lower=-3.14159 upper=3.14159 effort=0.0 velocity=0.0
- added joint torso_rightleg: type revolute, parent torso, child rightleg, origin xyz=0.5 0.5 1 rpy=0 0 0, axis 0 1 0, limit lower=-3.14159 upper=3.14159 effort=0.0 velocity=0.0

Commit message: snake

File: body.urdf (robot description, URDF)
Before this commit: robot robot, 9 links, 8 joints
Links:
- removed link backleg
- removed link backleg2
- removed link frontleg
- removed link frontleg2
- removed link leftleg
- removed link leftleg2
- removed link rightleg
- removed link rightleg2
- removed link torso
- added link link0, mass 1; collision box size=0.9156867995178384 0.739347251431691 0.5716602112218419; visual box size=0.9156867995178384 0.739347251431691 0.5716602112218419
- added link link1, mass 1; collision box size=0.20133165251050347 0.3465504939280762 0.6059611124094011; visual box size=0.20133165251050347 0.3465504939280762 0.6059611124094011
- added link link2, mass 1; collision box size=0.9735318012785863 0.40980788046345745 0.5721905470090412; visual box size=0.9735318012785863 0.40980788046345745 0.5721905470090412
- added link link3, mass 1; collision box size=0.8851759037168065 0.6050346099158632 0.5568431652519135; visual box size=0.8851759037168065 0.6050346099158632 0.5568431652519135
- added link link4, mass 1; collision box size=0.7068588011594938 0.23310842990509972 0.6746273165550472; visual box size=0.7068588011594938 0.23310842990509972 0.6746273165550472
- added link link5, mass 1; collision box size=0.869054692869264 0.3780598614737965 0.688968491745472; visual box size=0.869054692869264 0.3780598614737965 0.688968491745472
Joints:
- removed joint backleg_backleg2
- removed joint frontleg_frontleg2
- removed joint leftleg_leftleg2
- removed joint rightleg_rightleg2
- removed joint torso_backleg
- removed joint torso_frontleg
- removed joint torso_leftleg
- removed joint torso_rightleg
- added joint link0_link1: type revolute, parent link0, child link1, origin xyz=0.9156867995178384 0 0.3811068074812279 rpy=0 0 0, axis 0 1 0, limit lower=-3.14159 upper=3.14159 effort=0.0 velocity=0.0
- added joint link1_link2: type revolute, parent link1, child link2, origin xyz=0.20133165251050347 0 0.022867267458372864 rpy=0 0 0, axis 0 1 0, limit lower=-3.14159 upper=3.14159 effort=0.0 velocity=0.0
- added joint link2_link3: type revolute, parent link2, child link3, origin xyz=0.9735318012785863 0 -0.022513710266906628 rpy=0 0 0, axis 0 0 1, limit lower=-3.14159 upper=3.14159 effort=0.0 velocity=0.0
- added joint link3_link4: type revolute, parent link3, child link4, origin xyz=0.8851759037168065 0 -0.010231587838085143 rpy=0 0 0, axis 0 0 1, limit lower=-3.14159 upper=3.14159 effort=0.0 velocity=0.0
- added joint link4_link5: type revolute, parent link4, child link5, origin xyz=0.7068588011594938 0 0.07852276753542248 rpy=0 0 0, axis 0 0 1, limit lower=-3.14159 upper=3.14159 effort=0.0 velocity=0.0

Commit message: assignment7

File: body.urdf (robot description, URDF)
Before this commit: robot robot, 6 links, 5 joints
Links:
- removed link link0
- removed link link1
- removed link link2
- removed link link3
- removed link link4
- removed link link5
- added link LeftLowerLeg0, mass 1; collision box size=0.3689672379282213 0.14567881872974955 0.3701811501665392; visual box size=0.3689672379282213 0.14567881872974955 0.3701811501665392
- added link LeftLowerLeg1, mass 1; collision box size=0.3689672379282213 0.14567881872974955 0.3701811501665392; visual box size=0.3689672379282213 0.14567881872974955 0.3701811501665392
- added link LeftLowerLeg2, mass 1; collision box size=0.3689672379282213 0.14567881872974955 0.3701811501665392; visual box size=0.3689672379282213 0.14567881872974955 0.3701811501665392
- added link LeftLowerLeg3, mass 1; collision box size=0.3689672379282213 0.14567881872974955 0.3701811501665392; visual box size=0.3689672379282213 0.14567881872974955 0.3701811501665392
- added link LeftUpperLeg0, mass 1; collision box size=0.26282609074363356 0.15033034977577814 0.29473531493888167; visual box size=0.26282609074363356 0.15033034977577814 0.29473531493888167
- added link LeftUpperLeg1, mass 1; collision box size=0.26282609074363356 0.15033034977577814 0.29473531493888167; visual box size=0.26282609074363356 0.15033034977577814 0.29473531493888167
- added link LeftUpperLeg2, mass 1; collision box size=0.26282609074363356 0.15033034977577814 0.29473531493888167; visual box size=0.26282609074363356 0.15033034977577814 0.29473531493888167
- added link LeftUpperLeg3, mass 1; collision box size=0.26282609074363356 0.15033034977577814 0.29473531493888167; visual box size=0.26282609074363356 0.15033034977577814 0.29473531493888167
- added link RightLowerLeg0, mass 1; collision box size=0.3689672379282213 0.14567881872974955 0.3701811501665392; visual box size=0.3689672379282213 0.14567881872974955 0.3701811501665392
- added link RightLowerLeg1, mass 1; collision box size=0.3689672379282213 0.14567881872974955 0.3701811501665392; visual box size=0.3689672379282213 0.14567881872974955 0.3701811501665392
- added link RightLowerLeg2, mass 1; collision box size=0.3689672379282213 0.14567881872974955 0.3701811501665392; visual box size=0.3689672379282213 0.14567881872974955 0.3701811501665392
- added link RightLowerLeg3, mass 1; collision box size=0.3689672379282213 0.14567881872974955 0.3701811501665392; visual box size=0.3689672379282213 0.14567881872974955 0.3701811501665392
- added link RightUpperLeg0, mass 1; collision box size=0.26282609074363356 0.15033034977577814 0.29473531493888167; visual box size=0.26282609074363356 0.15033034977577814 0.29473531493888167
- added link RightUpperLeg1, mass 1; collision box size=0.26282609074363356 0.15033034977577814 0.29473531493888167; visual box size=0.26282609074363356 0.15033034977577814 0.29473531493888167
- added link RightUpperLeg2, mass 1; collision box size=0.26282609074363356 0.15033034977577814 0.29473531493888167; visual box size=0.26282609074363356 0.15033034977577814 0.29473531493888167
- added link RightUpperLeg3, mass 1; collision box size=0.26282609074363356 0.15033034977577814 0.29473531493888167; visual box size=0.26282609074363356 0.15033034977577814 0.29473531493888167
- added link body0, mass 1; collision box size=0.5189411367548277 0.35612537114724974 0.3415136925858484; visual box size=0.5189411367548277 0.35612537114724974 0.3415136925858484
- added link body1, mass 1; collision box size=0.5189411367548277 0.35612537114724974 0.3415136925858484; visual box size=0.5189411367548277 0.35612537114724974 0.3415136925858484
- added link body2, mass 1; collision box size=0.5189411367548277 0.35612537114724974 0.3415136925858484; visual box size=0.5189411367548277 0.35612537114724974 0.3415136925858484
- added link body3, mass 1; collision box size=0.5189411367548277 0.35612537114724974 0.3415136925858484; visual box size=0.5189411367548277 0.35612537114724974 0.3415136925858484
Joints:
- removed joint link0_link1
- removed joint link1_link2
- removed joint link2_link3
- removed joint link3_link4
- removed joint link4_link5
- added joint LeftUpperLeg0_LeftLowerLeg0: type revolute, parent LeftUpperLeg0, child LeftLowerLeg0, origin xyz=0 0.07516517488788907 -0.29473531493888167 rpy=0 0 0, axis 0 1 0, limit lower=-3.14159 upper=3.14159 effort=0.0 velocity=0.0
- added joint LeftUpperLeg1_LeftLowerLeg1: type revolute, parent LeftUpperLeg1, child LeftLowerLeg1, origin xyz=0 0.07516517488788907 -0.29473531493888167 rpy=0 0 0, axis 0 1 0, limit lower=-3.14159 upper=3.14159 effort=0.0 velocity=0.0
- added joint LeftUpperLeg2_LeftLowerLeg2: type revolute, parent LeftUpperLeg2, child LeftLowerLeg2, origin xyz=0.26282609074363356 0 0 rpy=0 0 0, axis 0 1 0, limit lower=-3.14159 upper=3.14159 effort=0.0 velocity=0.0
- added joint LeftUpperLeg3_LeftLowerLeg3: type revolute, parent LeftUpperLeg3, child LeftLowerLeg3, origin xyz=0 0.07516517488788907 -0.29473531493888167 rpy=0 0 0, axis 0 1 0, limit lower=-3.14159 upper=3.14159 effort=0.0 velocity=0.0
- added joint RightUpperLeg0_RightLowerLeg0: type revolute, parent RightUpperLeg0, child RightLowerLeg0, origin xyz=0 -0.07516517488788907 -0.29473531493888167 rpy=0 0 0, axis 0 1 0, limit lower=-3.14159 upper=3.14159 effort=0.0 velocity=0.0
- added joint RightUpperLeg1_RightLowerLeg1: type revolute, parent RightUpperLeg1, child RightLowerLeg1, origin xyz=0 -0.07516517488788907 -0.29473531493888167 rpy=0 0 0, axis 0 1 0, limit lower=-3.14159 upper=3.14159 effort=0.0 velocity=0.0
- added joint RightUpperLeg2_RightLowerLeg2: type revolute, parent RightUpperLeg2, child RightLowerLeg2, origin xyz=0 -0.07516517488788907 -0.29473531493888167 rpy=0 0 0, axis 0 1 0, limit lower=-3.14159 upper=3.14159 effort=0.0 velocity=0.0
- added joint RightUpperLeg3_RightLowerLeg3: type revolute, parent RightUpperLeg3, child RightLowerLeg3, origin xyz=0 -0.07516517488788907 -0.29473531493888167 rpy=0 0 0, axis 0 1 0, limit lower=-3.14159 upper=3.14159 effort=0.0 velocity=0.0
- added joint body0_LeftUpperLeg0: type revolute, parent body0, child LeftUpperLeg0, origin xyz=0.25947056837741383 0.17806268557362487 0.6649164651054209 rpy=0 0 0, axis 0 1 0, limit lower=-3.14159 upper=3.14159 effort=0.0 velocity=0.0
- added joint body0_RightUpperLeg0: type revolute, parent body0, child RightUpperLeg0, origin xyz=0.25947056837741383 -0.17806268557362487 0.6649164651054209 rpy=0 0 0, axis 0 1 0, limit lower=-3.14159 upper=3.14159 effort=0.0 velocity=0.0
- added joint body0_body1: type revolute, parent body0, child body1, origin xyz=0.5189411367548277 0 0.6649164651054209 rpy=0 0 0, axis 0 1 0, limit lower=-3.14159 upper=3.14159 effort=0.0 velocity=0.0
- added joint body1_LeftUpperLeg1: type revolute, parent body1, child LeftUpperLeg1, origin xyz=0.25947056837741383 0.17806268557362487 0 rpy=0 0 0, axis 0 1 0, limit lower=-3.14159 upper=3.14159 effort=0.0 velocity=0.0
- added joint body1_RightUpperLeg1: type revolute, parent body1, child RightUpperLeg1, origin xyz=0.25947056837741383 -0.17806268557362487 0 rpy=0 0 0, axis 0 1 0, limit lower=-3.14159 upper=3.14159 effort=0.0 velocity=0.0
- added joint body1_body2: type revolute, parent body1, child body2, origin xyz=0.5189411367548277 0 0 rpy=0 0 0, axis 0 1 0, limit lower=-3.14159 upper=3.14159 effort=0.0 velocity=0.0
- added joint body2_LeftUpperLeg2: type revolute, parent body2, child LeftUpperLeg2, origin xyz=0.25947056837741383 0.17806268557362487 0 rpy=0 0 0, axis 0 1 0, limit lower=-3.14159 upper=3.14159 effort=0.0 velocity=0.0
- added joint body2_RightUpperLeg2: type revolute, parent body2, child RightUpperLeg2, origin xyz=0.25947056837741383 -0.17806268557362487 0 rpy=0 0 0, axis 0 1 0, limit lower=-3.14159 upper=3.14159 effort=0.0 velocity=0.0
- added joint body2_body3: type revolute, parent body2, child body3, origin xyz=0.5189411367548277 0 0 rpy=0 0 0, axis 0 1 0, limit lower=-3.14159 upper=3.14159 effort=0.0 velocity=0.0
- added joint body3_LeftUpperLeg3: type revolute, parent body3, child LeftUpperLeg3, origin xyz=0.25947056837741383 0.17806268557362487 0 rpy=0 0 0, axis 0 1 0, limit lower=-3.14159 upper=3.14159 effort=0.0 velocity=0.0
- added joint body3_RightUpperLeg3: type revolute, parent body3, child RightUpperLeg3, origin xyz=0.25947056837741383 -0.17806268557362487 0 rpy=0 0 0, axis 0 1 0, limit lower=-3.14159 upper=3.14159 effort=0.0 velocity=0.0
