Commit message: assignment8 refactor

File: data/body.urdf (robot description, URDF)
Before this commit: robot robot, 20 links, 19 joints
Links:
- link LeftLowerLeg0: geometry collision box size=0.17082150821334013 0.11943157712446245 0.5114295236138631; visual box size=0.17082150821334013 0.11943157712446245 0.5114295236138631
- link LeftLowerLeg1: geometry collision box size=0.17082150821334013 0.11943157712446245 0.5114295236138631; visual box size=0.17082150821334013 0.11943157712446245 0.5114295236138631
- link LeftLowerLeg2: geometry collision box size=0.17082150821334013 0.11943157712446245 0.5114295236138631; visual box size=0.17082150821334013 0.11943157712446245 0.5114295236138631
- link LeftLowerLeg3: geometry collision box size=0.17082150821334013 0.11943157712446245 0.5114295236138631; visual box size=0.17082150821334013 0.11943157712446245 0.5114295236138631
- link LeftUpperLeg0: geometry collision box size=0.17120846509695148 0.5159703259691859 0.10416367677759474; visual box size=0.17120846509695148 0.5159703259691859 0.10416367677759474
- link LeftUpperLeg1: geometry collision box size=0.17120846509695148 0.5159703259691859 0.10416367677759474; visual box size=0.17120846509695148 0.5159703259691859 0.10416367677759474
- link LeftUpperLeg2: geometry collision box size=0.17120846509695148 0.5159703259691859 0.10416367677759474; visual box size=0.17120846509695148 0.5159703259691859 0.10416367677759474
- link LeftUpperLeg3: geometry collision box size=0.17120846509695148 0.5159703259691859 0.10416367677759474; visual box size=0.17120846509695148 0.5159703259691859 0.10416367677759474
- link RightLowerLeg0: geometry collision box size=0.17082150821334013 0.11943157712446245 0.5114295236138631; visual box size=0.17082150821334013 0.11943157712446245 0.5114295236138631
- link RightLowerLeg1: geometry collision box size=0.17082150821334013 0.11943157712446245 0.5114295236138631; visual box size=0.17082150821334013 0.11943157712446245 0.5114295236138631
- link RightLowerLeg2: geometry collision box size=0.17082150821334013 0.11943157712446245 0.5114295236138631; visual box size=0.17082150821334013 0.11943157712446245 0.5114295236138631
- link RightLowerLeg3: geometry collision box size=0.17082150821334013 0.11943157712446245 0.5114295236138631; visual box size=0.17082150821334013 0.11943157712446245 0.5114295236138631
- link RightUpperLeg0: geometry collision box size=0.17120846509695148 0.5159703259691859 0.10416367677759474; visual box size=0.17120846509695148 0.5159703259691859 0.10416367677759474
- link RightUpperLeg1: geometry collision box size=0.17120846509695148 0.5159703259691859 0.10416367677759474; visual box size=0.17120846509695148 0.5159703259691859 0.10416367677759474
- link RightUpperLeg2: geometry collision box size=0.17120846509695148 0.5159703259691859 0.10416367677759474; visual box size=0.17120846509695148 0.5159703259691859 0.10416367677759474
- link RightUpperLeg3: geometry collision box size=0.17120846509695148 0.5159703259691859 0.10416367677759474; visual box size=0.17120846509695148 0.5159703259691859 0.10416367677759474
- link body0: geometry collision box size=0.28853732159667966 0.18947474420985577 0.15348019668864246; visual box size=0.28853732159667966 0.18947474420985577 0.15348019668864246
- link body1: geometry collision box size=0.28853732159667966 0.18947474420985577 0.15348019668864246; visual box size=0.28853732159667966 0.18947474420985577 0.15348019668864246
- link body2: geometry collision box size=0.28853732159667966 0.18947474420985577 0.15348019668864246; visual box size=0.28853732159667966 0.18947474420985577 0.15348019668864246
- link body3: geometry collision box size=0.28853732159667966 0.18947474420985577 0.15348019668864246; visual box size=0.28853732159667966 0.18947474420985577 0.15348019668864246
Joints:
- joint LeftUpperLeg0_LeftLowerLeg0: axis 0 1 0 -> 1 0 0 ; origin xyz=0 0.08367588856022462 -0.549210117954695 rpy=0 0 0 -> xyz=0 0.5159703259691859 -0.10416367677759474 rpy=0 0 0
- joint LeftUpperLeg1_LeftLowerLeg1: axis 0 1 0 -> 1 0 0 ; origin xyz=0 0.08367588856022462 -0.549210117954695 rpy=0 0 0 -> xyz=0 0.5159703259691859 -0.10416367677759474 rpy=0 0 0
- joint LeftUpperLeg2_LeftLowerLeg2: axis 0 1 0 -> 1 0 0 ; origin xyz=0.14243925208510708 0 0 rpy=0 0 0 -> xyz=0 0.5159703259691859 -0.10416367677759474 rpy=0 0 0
- joint LeftUpperLeg3_LeftLowerLeg3: axis 0 1 0 -> 1 0 0 ; origin xyz=0 0.08367588856022462 -0.549210117954695 rpy=0 0 0 -> xyz=0 0.5159703259691859 -0.10416367677759474 rpy=0 0 0
- joint RightUpperLeg0_RightLowerLeg0: axis 0 1 0 -> 1 0 0 ; origin xyz=0 -0.08367588856022462 -0.549210117954695 rpy=0 0 0 -> xyz=0 -0.5159703259691859 -0.10416367677759474 rpy=0 0 0
- joint RightUpperLeg1_RightLowerLeg1: axis 0 1 0 -> 1 0 0 ; origin xyz=0 -0.08367588856022462 -0.549210117954695 rpy=0 0 0 -> xyz=0 -0.5159703259691859 -0.10416367677759474 rpy=0 0 0
- joint RightUpperLeg2_RightLowerLeg2: axis 0 1 0 -> 1 0 0 ; origin xyz=0 -0.08367588856022462 -0.549210117954695 rpy=0 0 0 -> xyz=0 -0.5159703259691859 -0.10416367677759474 rpy=0 0 0
- joint RightUpperLeg3_RightLowerLeg3: axis 0 1 0 -> 1 0 0 ; origin xyz=0 -0.08367588856022462 -0.549210117954695 rpy=0 0 0 -> xyz=0 -0.5159703259691859 -0.10416367677759474 rpy=0 0 0
- joint body0_LeftUpperLeg0: axis 0 1 0 -> 1 0 0 ; origin xyz=0.2639052370839119 0.2022589003624931 0.751789692233009 rpy=0 0 0 -> xyz=0.14426866079833983 0.09473737210492789 0.6155932003914578 rpy=0 0 0
- joint body0_RightUpperLeg0: axis 0 1 0 -> 1 0 0 ; origin xyz=0.2639052370839119 -0.2022589003624931 0.751789692233009 rpy=0 0 0 -> xyz=0.14426866079833983 -0.09473737210492789 0.6155932003914578 rpy=0 0 0
- joint body0_body1: axis 0 1 0 -> 0 0 1; origin xyz=0.5278104741678238 0 0.751789692233009 rpy=0 0 0 -> xyz=0.28853732159667966 0 0.6155932003914578 rpy=0 0 0
- joint body1_LeftUpperLeg1: axis 0 1 0 -> 1 0 0 ; origin xyz=0.2639052370839119 0.2022589003624931 0 rpy=0 0 0 -> xyz=0.14426866079833983 0.09473737210492789 0 rpy=0 0 0
- joint body1_RightUpperLeg1: axis 0 1 0 -> 1 0 0 ; origin xyz=0.2639052370839119 -0.2022589003624931 0 rpy=0 0 0 -> xyz=0.14426866079833983 -0.09473737210492789 0 rpy=0 0 0
- joint body1_body2: axis 0 1 0 -> 0 0 1; origin xyz=0.5278104741678238 0 0 rpy=0 0 0 -> xyz=0.28853732159667966 0 0 rpy=0 0 0
- joint body2_LeftUpperLeg2: axis 0 1 0 -> 1 0 0 ; origin xyz=0.2639052370839119 0.2022589003624931 0 rpy=0 0 0 -> xyz=0.14426866079833983 0.09473737210492789 0 rpy=0 0 0
- joint body2_RightUpperLeg2: axis 0 1 0 -> 1 0 0 ; origin xyz=0.2639052370839119 -0.2022589003624931 0 rpy=0 0 0 -> xyz=0.14426866079833983 -0.09473737210492789 0 rpy=0 0 0
- joint body2_body3: axis 0 1 0 -> 0 0 1; origin xyz=0.5278104741678238 0 0 rpy=0 0 0 -> xyz=0.28853732159667966 0 0 rpy=0 0 0
- joint body3_LeftUpperLeg3: axis 0 1 0 -> 1 0 0 ; origin xyz=0.2639052370839119 0.2022589003624931 0 rpy=0 0 0 -> xyz=0.14426866079833983 0.09473737210492789 0 rpy=0 0 0
- joint body3_RightUpperLeg3: axis 0 1 0 -> 1 0 0 ; origin xyz=0.2639052370839119 -0.2022589003624931 0 rpy=0 0 0 -> xyz=0.14426866079833983 -0.09473737210492789 0 rpy=0 0 0
