Commit message: final data

File: data/seed3/body.urdf (robot description, URDF)
Before this commit: robot robot, 20 links, 19 joints
Links:
- link LeftLowerLeg0: geometry collision box size=0.30779012326207505 0.23377013287434628 0.381170231505061; visual box size=0.30779012326207505 0.23377013287434628 0.381170231505061
- link LeftLowerLeg1: geometry collision box size=0.30779012326207505 0.23377013287434628 0.381170231505061; visual box size=0.30779012326207505 0.23377013287434628 0.381170231505061
- link LeftLowerLeg2: geometry collision box size=0.30779012326207505 0.23377013287434628 0.381170231505061; visual box size=0.30779012326207505 0.23377013287434628 0.381170231505061
- link LeftLowerLeg3: geometry collision box size=0.30779012326207505 0.23377013287434628 0.381170231505061; visual box size=0.30779012326207505 0.23377013287434628 0.381170231505061
- link LeftUpperLeg0: geometry collision box size=0.3281735454530538 0.1191309396491238 0.6205205779046914; visual box size=0.3281735454530538 0.1191309396491238 0.6205205779046914
- link LeftUpperLeg1: geometry collision box size=0.3281735454530538 0.1191309396491238 0.6205205779046914; visual box size=0.3281735454530538 0.1191309396491238 0.6205205779046914
- link LeftUpperLeg2: geometry collision box size=0.3281735454530538 0.1191309396491238 0.6205205779046914; visual box size=0.3281735454530538 0.1191309396491238 0.6205205779046914
- link LeftUpperLeg3: geometry collision box size=0.3281735454530538 0.1191309396491238 0.6205205779046914; visual box size=0.3281735454530538 0.1191309396491238 0.6205205779046914
- link RightLowerLeg0: geometry collision box size=0.30779012326207505 0.23377013287434628 0.381170231505061; visual box size=0.30779012326207505 0.23377013287434628 0.381170231505061
- link RightLowerLeg1: geometry collision box size=0.30779012326207505 0.23377013287434628 0.381170231505061; visual box size=0.30779012326207505 0.23377013287434628 0.381170231505061
- link RightLowerLeg2: geometry collision box size=0.30779012326207505 0.23377013287434628 0.381170231505061; visual box size=0.30779012326207505 0.23377013287434628 0.381170231505061
- link RightLowerLeg3: geometry collision box size=0.30779012326207505 0.23377013287434628 0.381170231505061; visual box size=0.30779012326207505 0.23377013287434628 0.381170231505061
- link RightUpperLeg0: geometry collision box size=0.3281735454530538 0.1191309396491238 0.6205205779046914; visual box size=0.3281735454530538 0.1191309396491238 0.6205205779046914
- link RightUpperLeg1: geometry collision box size=0.3281735454530538 0.1191309396491238 0.6205205779046914; visual box size=0.3281735454530538 0.1191309396491238 0.6205205779046914
- link RightUpperLeg2: geometry collision box size=0.3281735454530538 0.1191309396491238 0.6205205779046914; visual box size=0.3281735454530538 0.1191309396491238 0.6205205779046914
- link RightUpperLeg3: geometry collision box size=0.3281735454530538 0.1191309396491238 0.6205205779046914; visual box size=0.3281735454530538 0.1191309396491238 0.6205205779046914
- link body0: geometry collision box size=0.5056138779147621 0.28706236576520683 0.13760005610216533; visual box size=0.5056138779147621 0.28706236576520683 0.13760005610216533
- link body1: geometry collision box size=0.5056138779147621 0.28706236576520683 0.13760005610216533; visual box size=0.5056138779147621 0.28706236576520683 0.13760005610216533
- link body2: geometry collision box size=0.5056138779147621 0.28706236576520683 0.13760005610216533; visual box size=0.5056138779147621 0.28706236576520683 0.13760005610216533
- link body3: geometry collision box size=0.5056138779147621 0.28706236576520683 0.13760005610216533; visual box size=0.5056138779147621 0.28706236576520683 0.13760005610216533
Joints:
- joint LeftUpperLeg0_LeftLowerLeg0: origin xyz=0 0.07031377244518003 -0.2680034893263093 rpy=0 0 0 -> xyz=0 0.0595654698245619 -0.6205205779046914 rpy=0 0 0
- joint LeftUpperLeg1_LeftLowerLeg1: origin xyz=0 0.07031377244518003 -0.2680034893263093 rpy=0 0 0 -> xyz=0 0.0595654698245619 -0.6205205779046914 rpy=0 0 0
- joint LeftUpperLeg2_LeftLowerLeg2: origin xyz=0.31046453395357687 0 0 rpy=0 0 0 -> xyz=0.3281735454530538 0 0 rpy=0 0 0
- joint LeftUpperLeg3_LeftLowerLeg3: origin xyz=0 0.07031377244518003 -0.2680034893263093 rpy=0 0 0 -> xyz=0 0.0595654698245619 -0.6205205779046914 rpy=0 0 0
- joint RightUpperLeg0_RightLowerLeg0: origin xyz=0 -0.07031377244518003 -0.2680034893263093 rpy=0 0 0 -> xyz=0 -0.0595654698245619 -0.6205205779046914 rpy=0 0 0
- joint RightUpperLeg1_RightLowerLeg1: origin xyz=0 -0.07031377244518003 -0.2680034893263093 rpy=0 0 0 -> xyz=0 -0.0595654698245619 -0.6205205779046914 rpy=0 0 0
- joint RightUpperLeg2_RightLowerLeg2: origin xyz=0 -0.07031377244518003 -0.2680034893263093 rpy=0 0 0 -> xyz=0 -0.0595654698245619 -0.6205205779046914 rpy=0 0 0
- joint RightUpperLeg3_RightLowerLeg3: origin xyz=0 -0.07031377244518003 -0.2680034893263093 rpy=0 0 0 -> xyz=0 -0.0595654698245619 -0.6205205779046914 rpy=0 0 0
- joint body0_LeftUpperLeg0: origin xyz=0.14348779535100614 0.2336645100987486 0.9396569410464768 rpy=0 0 0 -> xyz=0.25280693895738104 0.14353118288260341 1.0016908094097525 rpy=0 0 0
- joint body0_RightUpperLeg0: origin xyz=0.14348779535100614 -0.2336645100987486 0.9396569410464768 rpy=0 0 0 -> xyz=0.25280693895738104 -0.14353118288260341 1.0016908094097525 rpy=0 0 0
- joint body0_body1: origin xyz=0.2869755907020123 0 0.9396569410464768 rpy=0 0 0 -> xyz=0.5056138779147621 0 1.0016908094097525 rpy=0 0 0
- joint body1_LeftUpperLeg1: origin xyz=0.14348779535100614 0.2336645100987486 0 rpy=0 0 0 -> xyz=0.25280693895738104 0.14353118288260341 0 rpy=0 0 0
- joint body1_RightUpperLeg1: origin xyz=0.14348779535100614 -0.2336645100987486 0 rpy=0 0 0 -> xyz=0.25280693895738104 -0.14353118288260341 0 rpy=0 0 0
- joint body1_body2: origin xyz=0.2869755907020123 0 0 rpy=0 0 0 -> xyz=0.5056138779147621 0 0 rpy=0 0 0
- joint body2_LeftUpperLeg2: origin xyz=0.14348779535100614 0.2336645100987486 0 rpy=0 0 0 -> xyz=0.25280693895738104 0.14353118288260341 0 rpy=0 0 0
- joint body2_RightUpperLeg2: origin xyz=0.14348779535100614 -0.2336645100987486 0 rpy=0 0 0 -> xyz=0.25280693895738104 -0.14353118288260341 0 rpy=0 0 0
- joint body2_body3: origin xyz=0.2869755907020123 0 0 rpy=0 0 0 -> xyz=0.5056138779147621 0 0 rpy=0 0 0
- joint body3_LeftUpperLeg3: origin xyz=0.14348779535100614 0.2336645100987486 0 rpy=0 0 0 -> xyz=0.25280693895738104 0.14353118288260341 0 rpy=0 0 0
- joint body3_RightUpperLeg3: origin xyz=0.14348779535100614 -0.2336645100987486 0 rpy=0 0 0 -> xyz=0.25280693895738104 -0.14353118288260341 0 rpy=0 0 0

File: data/seed4/body.urdf (robot description, URDF)
Before this commit: robot robot, 20 links, 19 joints
Links:
- link LeftLowerLeg0: geometry collision box size=0.3709535571220328 0.2898889313177383 0.2025795742783139; visual box size=0.3709535571220328 0.2898889313177383 0.2025795742783139
- link LeftLowerLeg1: geometry collision box size=0.3709535571220328 0.2898889313177383 0.2025795742783139; visual box size=0.3709535571220328 0.2898889313177383 0.2025795742783139
- link LeftLowerLeg2: geometry collision box size=0.3709535571220328 0.2898889313177383 0.2025795742783139; visual box size=0.3709535571220328 0.2898889313177383 0.2025795742783139
- link LeftLowerLeg3: geometry collision box size=0.3709535571220328 0.2898889313177383 0.2025795742783139; visual box size=0.3709535571220328 0.2898889313177383 0.2025795742783139
- link LeftUpperLeg0: geometry collision box size=0.14243925208510708 0.16735177712044924 0.549210117954695; visual box size=0.14243925208510708 0.16735177712044924 0.549210117954695
- link LeftUpperLeg1: geometry collision box size=0.14243925208510708 0.16735177712044924 0.549210117954695; visual box size=0.14243925208510708 0.16735177712044924 0.549210117954695
- link LeftUpperLeg2: geometry collision box size=0.14243925208510708 0.16735177712044924 0.549210117954695; visual box size=0.14243925208510708 0.16735177712044924 0.549210117954695
- link LeftUpperLeg3: geometry collision box size=0.14243925208510708 0.16735177712044924 0.549210117954695; visual box size=0.14243925208510708 0.16735177712044924 0.549210117954695
- link RightLowerLeg0: geometry collision box size=0.3709535571220328 0.2898889313177383 0.2025795742783139; visual box size=0.3709535571220328 0.2898889313177383 0.2025795742783139
- link RightLowerLeg1: geometry collision box size=0.3709535571220328 0.2898889313177383 0.2025795742783139; visual box size=0.3709535571220328 0.2898889313177383 0.2025795742783139
- link RightLowerLeg2: geometry collision box size=0.3709535571220328 0.2898889313177383 0.2025795742783139; visual box size=0.3709535571220328 0.2898889313177383 0.2025795742783139
- link RightLowerLeg3: geometry collision box size=0.3709535571220328 0.2898889313177383 0.2025795742783139; visual box size=0.3709535571220328 0.2898889313177383 0.2025795742783139
- link RightUpperLeg0: geometry collision box size=0.14243925208510708 0.16735177712044924 0.549210117954695; visual box size=0.14243925208510708 0.16735177712044924 0.549210117954695
- link RightUpperLeg1: geometry collision box size=0.14243925208510708 0.16735177712044924 0.549210117954695; visual box size=0.14243925208510708 0.16735177712044924 0.549210117954695
- link RightUpperLeg2: geometry collision box size=0.14243925208510708 0.16735177712044924 0.549210117954695; visual box size=0.14243925208510708 0.16735177712044924 0.549210117954695
- link RightUpperLeg3: geometry collision box size=0.14243925208510708 0.16735177712044924 0.549210117954695; visual box size=0.14243925208510708 0.16735177712044924 0.549210117954695
- link body0: geometry collision box size=0.5278104741678238 0.4045178007249862 0.3987781026068683; visual box size=0.5278104741678238 0.4045178007249862 0.3987781026068683
- link body1: geometry collision box size=0.5278104741678238 0.4045178007249862 0.3987781026068683; visual box size=0.5278104741678238 0.4045178007249862 0.3987781026068683
- link body2: geometry collision box size=0.5278104741678238 0.4045178007249862 0.3987781026068683; visual box size=0.5278104741678238 0.4045178007249862 0.3987781026068683
- link body3: geometry collision box size=0.5278104741678238 0.4045178007249862 0.3987781026068683; visual box size=0.5278104741678238 0.4045178007249862 0.3987781026068683
Joints:
- joint LeftUpperLeg0_LeftLowerLeg0: origin xyz=0 0.07031377244518003 -0.2680034893263093 rpy=0 0 0 -> xyz=0 0.08367588856022462 -0.549210117954695 rpy=0 0 0
- joint LeftUpperLeg1_LeftLowerLeg1: origin xyz=0 0.07031377244518003 -0.2680034893263093 rpy=0 0 0 -> xyz=0 0.08367588856022462 -0.549210117954695 rpy=0 0 0
- joint LeftUpperLeg2_LeftLowerLeg2: origin xyz=0.31046453395357687 0 0 rpy=0 0 0 -> xyz=0.14243925208510708 0 0 rpy=0 0 0
- joint LeftUpperLeg3_LeftLowerLeg3: origin xyz=0 0.07031377244518003 -0.2680034893263093 rpy=0 0 0 -> xyz=0 0.08367588856022462 -0.549210117954695 rpy=0 0 0
- joint RightUpperLeg0_RightLowerLeg0: origin xyz=0 -0.07031377244518003 -0.2680034893263093 rpy=0 0 0 -> xyz=0 -0.08367588856022462 -0.549210117954695 rpy=0 0 0
- joint RightUpperLeg1_RightLowerLeg1: origin xyz=0 -0.07031377244518003 -0.2680034893263093 rpy=0 0 0 -> xyz=0 -0.08367588856022462 -0.549210117954695 rpy=0 0 0
- joint RightUpperLeg2_RightLowerLeg2: origin xyz=0 -0.07031377244518003 -0.2680034893263093 rpy=0 0 0 -> xyz=0 -0.08367588856022462 -0.549210117954695 rpy=0 0 0
- joint RightUpperLeg3_RightLowerLeg3: origin xyz=0 -0.07031377244518003 -0.2680034893263093 rpy=0 0 0 -> xyz=0 -0.08367588856022462 -0.549210117954695 rpy=0 0 0
- joint body0_LeftUpperLeg0: origin xyz=0.14348779535100614 0.2336645100987486 0.9396569410464768 rpy=0 0 0 -> xyz=0.2639052370839119 0.2022589003624931 0.751789692233009 rpy=0 0 0
- joint body0_RightUpperLeg0: origin xyz=0.14348779535100614 -0.2336645100987486 0.9396569410464768 rpy=0 0 0 -> xyz=0.2639052370839119 -0.2022589003624931 0.751789692233009 rpy=0 0 0
- joint body0_body1: origin xyz=0.2869755907020123 0 0.9396569410464768 rpy=0 0 0 -> xyz=0.5278104741678238 0 0.751789692233009 rpy=0 0 0
- joint body1_LeftUpperLeg1: origin xyz=0.14348779535100614 0.2336645100987486 0 rpy=0 0 0 -> xyz=0.2639052370839119 0.2022589003624931 0 rpy=0 0 0
- joint body1_RightUpperLeg1: origin xyz=0.14348779535100614 -0.2336645100987486 0 rpy=0 0 0 -> xyz=0.2639052370839119 -0.2022589003624931 0 rpy=0 0 0
- joint body1_body2: origin xyz=0.2869755907020123 0 0 rpy=0 0 0 -> xyz=0.5278104741678238 0 0 rpy=0 0 0
- joint body2_LeftUpperLeg2: origin xyz=0.14348779535100614 0.2336645100987486 0 rpy=0 0 0 -> xyz=0.2639052370839119 0.2022589003624931 0 rpy=0 0 0
- joint body2_RightUpperLeg2: origin xyz=0.14348779535100614 -0.2336645100987486 0 rpy=0 0 0 -> xyz=0.2639052370839119 -0.2022589003624931 0 rpy=0 0 0
- joint body2_body3: origin xyz=0.2869755907020123 0 0 rpy=0 0 0 -> xyz=0.5278104741678238 0 0 rpy=0 0 0
- joint body3_LeftUpperLeg3: origin xyz=0.14348779535100614 0.2336645100987486 0 rpy=0 0 0 -> xyz=0.2639052370839119 0.2022589003624931 0 rpy=0 0 0
- joint body3_RightUpperLeg3: origin xyz=0.14348779535100614 -0.2336645100987486 0 rpy=0 0 0 -> xyz=0.2639052370839119 -0.2022589003624931 0 rpy=0 0 0

File: data/seed5/body.urdf (robot description, URDF)
Before this commit: robot robot, 20 links, 19 joints
Links:
- link LeftLowerLeg0: geometry collision box size=0.1563163685983755 0.12422238062946248 0.569220148099485; visual box size=0.1563163685983755 0.12422238062946248 0.569220148099485
- link LeftLowerLeg1: geometry collision box size=0.1563163685983755 0.12422238062946248 0.569220148099485; visual box size=0.1563163685983755 0.12422238062946248 0.569220148099485
- link LeftLowerLeg2: geometry collision box size=0.1563163685983755 0.12422238062946248 0.569220148099485; visual box size=0.1563163685983755 0.12422238062946248 0.569220148099485
- link LeftLowerLeg3: geometry collision box size=0.1563163685983755 0.12422238062946248 0.569220148099485; visual box size=0.1563163685983755 0.12422238062946248 0.569220148099485
- link LeftUpperLeg0: geometry collision box size=0.3297723569440947 0.255525396361883 0.348400250788111; visual box size=0.3297723569440947 0.255525396361883 0.348400250788111
- link LeftUpperLeg1: geometry collision box size=0.3297723569440947 0.255525396361883 0.348400250788111; visual box size=0.3297723569440947 0.255525396361883 0.348400250788111
- link LeftUpperLeg2: geometry collision box size=0.3297723569440947 0.255525396361883 0.348400250788111; visual box size=0.3297723569440947 0.255525396361883 0.348400250788111
- link LeftUpperLeg3: geometry collision box size=0.3297723569440947 0.255525396361883 0.348400250788111; visual box size=0.3297723569440947 0.255525396361883 0.348400250788111
- link RightLowerLeg0: geometry collision box size=0.1563163685983755 0.12422238062946248 0.569220148099485; visual box size=0.1563163685983755 0.12422238062946248 0.569220148099485
- link RightLowerLeg1: geometry collision box size=0.1563163685983755 0.12422238062946248 0.569220148099485; visual box size=0.1563163685983755 0.12422238062946248 0.569220148099485
- link RightLowerLeg2: geometry collision box size=0.1563163685983755 0.12422238062946248 0.569220148099485; visual box size=0.1563163685983755 0.12422238062946248 0.569220148099485
- link RightLowerLeg3: geometry collision box size=0.1563163685983755 0.12422238062946248 0.569220148099485; visual box size=0.1563163685983755 0.12422238062946248 0.569220148099485
- link RightUpperLeg0: geometry collision box size=0.3297723569440947 0.255525396361883 0.348400250788111; visual box size=0.3297723569440947 0.255525396361883 0.348400250788111
- link RightUpperLeg1: geometry collision box size=0.3297723569440947 0.255525396361883 0.348400250788111; visual box size=0.3297723569440947 0.255525396361883 0.348400250788111
- link RightUpperLeg2: geometry collision box size=0.3297723569440947 0.255525396361883 0.348400250788111; visual box size=0.3297723569440947 0.255525396361883 0.348400250788111
- link RightUpperLeg3: geometry collision box size=0.3297723569440947 0.255525396361883 0.348400250788111; visual box size=0.3297723569440947 0.255525396361883 0.348400250788111
- link body0: geometry collision box size=0.5593054539689608 0.3442055943974146 0.40587193145132283; visual box size=0.5593054539689608 0.3442055943974146 0.40587193145132283
- link body1: geometry collision box size=0.5593054539689608 0.3442055943974146 0.40587193145132283; visual box size=0.5593054539689608 0.3442055943974146 0.40587193145132283
- link body2: geometry collision box size=0.5593054539689608 0.3442055943974146 0.40587193145132283; visual box size=0.5593054539689608 0.3442055943974146 0.40587193145132283
- link body3: geometry collision box size=0.5593054539689608 0.3442055943974146 0.40587193145132283; visual box size=0.5593054539689608 0.3442055943974146 0.40587193145132283
Joints:
- joint LeftUpperLeg0_LeftLowerLeg0: origin xyz=0 0.07031377244518003 -0.2680034893263093 rpy=0 0 0 -> xyz=0 0.1277626981809415 -0.348400250788111 rpy=0 0 0
- joint LeftUpperLeg1_LeftLowerLeg1: origin xyz=0 0.07031377244518003 -0.2680034893263093 rpy=0 0 0 -> xyz=0 0.1277626981809415 -0.348400250788111 rpy=0 0 0
- joint LeftUpperLeg2_LeftLowerLeg2: origin xyz=0.31046453395357687 0 0 rpy=0 0 0 -> xyz=0.3297723569440947 0 0 rpy=0 0 0
- joint LeftUpperLeg3_LeftLowerLeg3: origin xyz=0 0.07031377244518003 -0.2680034893263093 rpy=0 0 0 -> xyz=0 0.1277626981809415 -0.348400250788111 rpy=0 0 0
- joint RightUpperLeg0_RightLowerLeg0: origin xyz=0 -0.07031377244518003 -0.2680034893263093 rpy=0 0 0 -> xyz=0 -0.1277626981809415 -0.348400250788111 rpy=0 0 0
- joint RightUpperLeg1_RightLowerLeg1: origin xyz=0 -0.07031377244518003 -0.2680034893263093 rpy=0 0 0 -> xyz=0 -0.1277626981809415 -0.348400250788111 rpy=0 0 0
- joint RightUpperLeg2_RightLowerLeg2: origin xyz=0 -0.07031377244518003 -0.2680034893263093 rpy=0 0 0 -> xyz=0 -0.1277626981809415 -0.348400250788111 rpy=0 0 0
- joint RightUpperLeg3_RightLowerLeg3: origin xyz=0 -0.07031377244518003 -0.2680034893263093 rpy=0 0 0 -> xyz=0 -0.1277626981809415 -0.348400250788111 rpy=0 0 0
- joint body0_LeftUpperLeg0: origin xyz=0.14348779535100614 0.2336645100987486 0.9396569410464768 rpy=0 0 0 -> xyz=0.2796527269844804 0.1721027971987073 0.917620398887596 rpy=0 0 0
- joint body0_RightUpperLeg0: origin xyz=0.14348779535100614 -0.2336645100987486 0.9396569410464768 rpy=0 0 0 -> xyz=0.2796527269844804 -0.1721027971987073 0.917620398887596 rpy=0 0 0
- joint body0_body1: origin xyz=0.2869755907020123 0 0.9396569410464768 rpy=0 0 0 -> xyz=0.5593054539689608 0 0.917620398887596 rpy=0 0 0
- joint body1_LeftUpperLeg1: origin xyz=0.14348779535100614 0.2336645100987486 0 rpy=0 0 0 -> xyz=0.2796527269844804 0.1721027971987073 0 rpy=0 0 0
- joint body1_RightUpperLeg1: origin xyz=0.14348779535100614 -0.2336645100987486 0 rpy=0 0 0 -> xyz=0.2796527269844804 -0.1721027971987073 0 rpy=0 0 0
- joint body1_body2: origin xyz=0.2869755907020123 0 0 rpy=0 0 0 -> xyz=0.5593054539689608 0 0 rpy=0 0 0
- joint body2_LeftUpperLeg2: origin xyz=0.14348779535100614 0.2336645100987486 0 rpy=0 0 0 -> xyz=0.2796527269844804 0.1721027971987073 0 rpy=0 0 0
- joint body2_RightUpperLeg2: origin xyz=0.14348779535100614 -0.2336645100987486 0 rpy=0 0 0 -> xyz=0.2796527269844804 -0.1721027971987073 0 rpy=0 0 0
- joint body2_body3: origin xyz=0.2869755907020123 0 0 rpy=0 0 0 -> xyz=0.5593054539689608 0 0 rpy=0 0 0
- joint body3_LeftUpperLeg3: origin xyz=0.14348779535100614 0.2336645100987486 0 rpy=0 0 0 -> xyz=0.2796527269844804 0.1721027971987073 0 rpy=0 0 0
- joint body3_RightUpperLeg3: origin xyz=0.14348779535100614 -0.2336645100987486 0 rpy=0 0 0 -> xyz=0.2796527269844804 -0.1721027971987073 0 rpy=0 0 0
