Commit message: final data

File: data/seed6/body.urdf (robot description, URDF)
Before this commit: robot robot, 20 links, 19 joints
Links:
- link LeftLowerLeg0: geometry collision box size=0.12545237978767 0.16698507980240057 0.3089451097583441; visual box size=0.12545237978767 0.16698507980240057 0.3089451097583441
- link LeftLowerLeg1: geometry collision box size=0.12545237978767 0.16698507980240057 0.3089451097583441; visual box size=0.12545237978767 0.16698507980240057 0.3089451097583441
- link LeftLowerLeg2: geometry collision box size=0.12545237978767 0.16698507980240057 0.3089451097583441; visual box size=0.12545237978767 0.16698507980240057 0.3089451097583441
- link LeftLowerLeg3: geometry collision box size=0.12545237978767 0.16698507980240057 0.3089451097583441; visual box size=0.12545237978767 0.16698507980240057 0.3089451097583441
- link LeftUpperLeg0: geometry collision box size=0.28494298244073635 0.2327531513741691 0.48797617601165233; visual box size=0.28494298244073635 0.2327531513741691 0.48797617601165233
- link LeftUpperLeg1: geometry collision box size=0.28494298244073635 0.2327531513741691 0.48797617601165233; visual box size=0.28494298244073635 0.2327531513741691 0.48797617601165233
- link LeftUpperLeg2: geometry collision box size=0.28494298244073635 0.2327531513741691 0.48797617601165233; visual box size=0.28494298244073635 0.2327531513741691 0.48797617601165233
- link LeftUpperLeg3: geometry collision box size=0.28494298244073635 0.2327531513741691 0.48797617601165233; visual box size=0.28494298244073635 0.2327531513741691 0.48797617601165233
- link RightLowerLeg0: geometry collision box size=0.12545237978767 0.16698507980240057 0.3089451097583441; visual box size=0.12545237978767 0.16698507980240057 0.3089451097583441
- link RightLowerLeg1: geometry collision box size=0.12545237978767 0.16698507980240057 0.3089451097583441; visual box size=0.12545237978767 0.16698507980240057 0.3089451097583441
- link RightLowerLeg2: geometry collision box size=0.12545237978767 0.16698507980240057 0.3089451097583441; visual box size=0.12545237978767 0.16698507980240057 0.3089451097583441
- link RightLowerLeg3: geometry collision box size=0.12545237978767 0.16698507980240057 0.3089451097583441; visual box size=0.12545237978767 0.16698507980240057 0.3089451097583441
- link RightUpperLeg0: geometry collision box size=0.28494298244073635 0.2327531513741691 0.48797617601165233; visual box size=0.28494298244073635 0.2327531513741691 0.48797617601165233
- link RightUpperLeg1: geometry collision box size=0.28494298244073635 0.2327531513741691 0.48797617601165233; visual box size=0.28494298244073635 0.2327531513741691 0.48797617601165233
- link RightUpperLeg2: geometry collision box size=0.28494298244073635 0.2327531513741691 0.48797617601165233; visual box size=0.28494298244073635 0.2327531513741691 0.48797617601165233
- link RightUpperLeg3: geometry collision box size=0.28494298244073635 0.2327531513741691 0.48797617601165233; visual box size=0.28494298244073635 0.2327531513741691 0.48797617601165233
- link body0: geometry collision box size=0.4369173397073046 0.1739223465404308 0.27854763469251487; visual box size=0.4369173397073046 0.1739223465404308 0.27854763469251487
- link body1: geometry collision box size=0.4369173397073046 0.1739223465404308 0.27854763469251487; visual box size=0.4369173397073046 0.1739223465404308 0.27854763469251487
- link body2: geometry collision box size=0.4369173397073046 0.1739223465404308 0.27854763469251487; visual box size=0.4369173397073046 0.1739223465404308 0.27854763469251487
- link body3: geometry collision box size=0.4369173397073046 0.1739223465404308 0.27854763469251487; visual box size=0.4369173397073046 0.1739223465404308 0.27854763469251487
Joints:
- joint LeftUpperLeg0_LeftLowerLeg0: origin xyz=0 0.07031377244518003 -0.2680034893263093 rpy=0 0 0 -> xyz=0 0.11637657568708455 -0.48797617601165233 rpy=0 0 0
- joint LeftUpperLeg1_LeftLowerLeg1: origin xyz=0 0.07031377244518003 -0.2680034893263093 rpy=0 0 0 -> xyz=0 0.11637657568708455 -0.48797617601165233 rpy=0 0 0
- joint LeftUpperLeg2_LeftLowerLeg2: origin xyz=0.31046453395357687 0 0 rpy=0 0 0 -> xyz=0.28494298244073635 0 0 rpy=0 0 0
- joint LeftUpperLeg3_LeftLowerLeg3: origin xyz=0 0.07031377244518003 -0.2680034893263093 rpy=0 0 0 -> xyz=0 0.11637657568708455 -0.48797617601165233 rpy=0 0 0
- joint RightUpperLeg0_RightLowerLeg0: origin xyz=0 -0.07031377244518003 -0.2680034893263093 rpy=0 0 0 -> xyz=0 -0.11637657568708455 -0.48797617601165233 rpy=0 0 0
- joint RightUpperLeg1_RightLowerLeg1: origin xyz=0 -0.07031377244518003 -0.2680034893263093 rpy=0 0 0 -> xyz=0 -0.11637657568708455 -0.48797617601165233 rpy=0 0 0
- joint RightUpperLeg2_RightLowerLeg2: origin xyz=0 -0.07031377244518003 -0.2680034893263093 rpy=0 0 0 -> xyz=0 -0.11637657568708455 -0.48797617601165233 rpy=0 0 0
- joint RightUpperLeg3_RightLowerLeg3: origin xyz=0 -0.07031377244518003 -0.2680034893263093 rpy=0 0 0 -> xyz=0 -0.11637657568708455 -0.48797617601165233 rpy=0 0 0
- joint body0_LeftUpperLeg0: origin xyz=0.14348779535100614 0.2336645100987486 0.9396569410464768 rpy=0 0 0 -> xyz=0.2184586698536523 0.0869611732702154 0.7969212857699964 rpy=0 0 0
- joint body0_RightUpperLeg0: origin xyz=0.14348779535100614 -0.2336645100987486 0.9396569410464768 rpy=0 0 0 -> xyz=0.2184586698536523 -0.0869611732702154 0.7969212857699964 rpy=0 0 0
- joint body0_body1: origin xyz=0.2869755907020123 0 0.9396569410464768 rpy=0 0 0 -> xyz=0.4369173397073046 0 0.7969212857699964 rpy=0 0 0
- joint body1_LeftUpperLeg1: origin xyz=0.14348779535100614 0.2336645100987486 0 rpy=0 0 0 -> xyz=0.2184586698536523 0.0869611732702154 0 rpy=0 0 0
- joint body1_RightUpperLeg1: origin xyz=0.14348779535100614 -0.2336645100987486 0 rpy=0 0 0 -> xyz=0.2184586698536523 -0.0869611732702154 0 rpy=0 0 0
- joint body1_body2: origin xyz=0.2869755907020123 0 0 rpy=0 0 0 -> xyz=0.4369173397073046 0 0 rpy=0 0 0
- joint body2_LeftUpperLeg2: origin xyz=0.14348779535100614 0.2336645100987486 0 rpy=0 0 0 -> xyz=0.2184586698536523 0.0869611732702154 0 rpy=0 0 0
- joint body2_RightUpperLeg2: origin xyz=0.14348779535100614 -0.2336645100987486 0 rpy=0 0 0 -> xyz=0.2184586698536523 -0.0869611732702154 0 rpy=0 0 0
- joint body2_body3: origin xyz=0.2869755907020123 0 0 rpy=0 0 0 -> xyz=0.4369173397073046 0 0 rpy=0 0 0
- joint body3_LeftUpperLeg3: origin xyz=0.14348779535100614 0.2336645100987486 0 rpy=0 0 0 -> xyz=0.2184586698536523 0.0869611732702154 0 rpy=0 0 0
- joint body3_RightUpperLeg3: origin xyz=0.14348779535100614 -0.2336645100987486 0 rpy=0 0 0 -> xyz=0.2184586698536523 -0.0869611732702154 0 rpy=0 0 0
